Commit message: Fix urdf.

File: resources/devq/urdf/devq.urdf (robot description, URDF)
Before this commit: robot alphadog_devq, 17 links, 16 joints
Links:
- link front_left_abad_link: geometry collision cylinder length=0.05 radius=0.04; visual mesh filename=../meshes/abad_link.STL scale=1 1 1
- link front_left_hip_link: geometry collision box size=0.04 0.025 0.12; visual mesh filename=../meshes/hip_link.STL scale=1 1 1
- link front_right_abad_link: geometry collision cylinder length=0.05 radius=0.04; visual mesh filename=../meshes/abad_link.STL scale=1 -1 1
- link front_right_hip_link: geometry collision box size=0.04 0.025 0.12; visual mesh filename=../meshes/hip_link.STL scale=1 -1 1
- link hind_left_abad_link: geometry collision cylinder length=0.05 radius=0.04; visual mesh filename=../meshes/abad_link.STL scale=-1 1 1
- link hind_left_hip_link: geometry collision box size=0.04 0.025 0.12; visual mesh filename=../meshes/hip_link.STL scale=1 1 1
- link hind_right_abad_link: geometry collision cylinder length=0.05 radius=0.04; visual mesh filename=../meshes/abad_link.STL scale=-1 -1 1
- link hind_right_hip_link: geometry collision box size=0.04 0.025 0.12; visual mesh filename=../meshes/hip_link.STL scale=1 -1 1
Joints:
- joint front_left_hip_joint: axis 0 -1 0 0 -> 0 -1 0
- joint front_right_hip_joint: axis 0 -1 0 0 -> 0 -1 0
- joint hind_left_hip_joint: axis 0 -1 0 0 -> 0 -1 0
- joint hind_right_hip_joint: axis 0 -1 0 0 -> 0 -1 0
